File: Eagle/funcgen.sch (EAGLE design)
At the start: 67 parts, among them IC1 AD9833, IC2 LD117ADT33TR, IC3 LM318D, IC6 LM318D, J1 DCJ0202, Q1 16MHz, Q2 ASFL1, U1 MICROCHIP_ATMEGA328PB-AUMICRO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, U3 TLV61048DBVR, X1 A1944-50

Commit message: Revised and Updated Schematic and Board
Changed schematic to multiple sheets with better organization. Board layout is redone entirely. Surface area is nearly cut in half from first design.
ISSUES: 1) need to verify / find the proper DC jack connector.
            2) need an 0805 inductor package. I believe I left enough space for it, but for now the footprint is entirely incorrect
Parts:
- removed C1, C10, C12, C13, C26, C4, C7, C8, C9: 0.1uF, rcl:C-EUC0805
- removed C22, C23: 22pF, rcl:C-EUC0805
- removed C25: 10uF, rcl:C-EUC0805
- removed IC2: LD117ADT33TR, v-reg:LD117ADT33TR
- removed IC3, IC6: LM318D, linear:LM318D
- removed JP1: (no value), jumper:JP2E
- removed JP2, JP4, LCD/I2C: (no value), jumper:JP1E
- removed JP3: (no value), jumper:JP4QE
- removed Q1: 16MHz, crystal:CRYSTALHC49UP
- removed R12, R13, R21, R22, R23, R27, R30, R31: 1k, rcl:R-EU_R0805
- removed R16, R17, R18, R19, R2, R20, R3: 10k, rcl:R-EU_R0805
- removed R26: 330, rcl:R-EU_R0805
- removed R4, R5: 1k3, rcl:R-EU_R0805
- removed U$1: AVR-ISP, AVR-ISP:AVR-ISP
- removed X1: A1944-50, con-coax:A1944-50
- added C14, C21, C28, C29, C31, C32, C33, C34, C35, C40: 0.1uF, rcl:C-EUC0805
- added C36, C37: 22pF, rcl:C-EUC0805
- added IC4, IC5: LM318D, linear:LM318D
- added JP5, JP7, LCD/I2C1, LCD_POW: (no value), jumper:JP1E
- added JP6: (no value), jumper:JP2E
- added JP8: (no value), jumper:JP4QE
- added Q3: 16MHz, crystal:CRYSTALHC49UP
- added R14, R15, R24, R32, R44, R8, R9: 10k, rcl:R-EU_R0805
- added R28, R29, R37, R38, R39, R41, R42, R43: 1k, rcl:R-EU_R0805
- added R40: 330, rcl:R-EU_R0805
- added R6, R7: 1k3, rcl:R-EU_R0805
- added U$2: AVR-ISP, AVR-ISP:AVR-ISP
- added U2: MICROCHIP_ATMEGA328PB-AUMICROCHIP_ATMEGA328PB-AU_0_0, Microchip - ATmega328PB-AU:MICROCHIP_ATMEGA328PB-AUMICROCHIP_ATMEGA328PB-AU_0_0
- C2, C3: value 0.1uF -> 10uF
- POT1K, POT50K: device jumper:JP2W -> jumper:JP2E
- U1: value MICROCHIP_ATMEGA328PB-AUMICROCHIP_ATMEGA328PB-AU_0_0 -> TLV1117-33IDCY; device Microchip - ATmega328PB-AU:MICROCHIP_ATMEGA328PB-AUMICROCHIP_ATMEGA328PB-AU_0_0 -> TLV1117-33IDCY:TLV1117-33IDCY
Connections:
- removed net N$1: IC3.+IN, R4.2
- removed net N$13: JP1.1, R2.2
- removed net N$14: JP1.3, R16.2
- removed net N$15: C23.1, Q1.2, U1.PB7(TOSC2/XTAL2)
- removed net N$16: R21.1, R27.2
- removed net N$17: R13.2, R27.1
- removed net N$18: JP3-1.2, R26.2
- removed net N$19: JP3-2.1, R22.2
- removed net N$2: IC3.-IN, POT50K.3, R5.2
- removed net N$20: JP3-2.2, R21.2
- removed net N$3: IC6.+IN, R19.1, R20.2
- removed net N$4: POT1K.2, R19.2
- removed net N$5: IC6.-IN, R17.1, R18.2
- removed net N$7: C22.2, Q1.1, U1.PB6(TOSC1/XTAL1)
- new net N$21: IC4.+IN, R6.2
- new net N$22: IC4.-IN, POT50K.3, R7.2
- new net N$24: IC5.+IN, R14.1, R15.2
- new net N$25: POT1K.2, R14.2
- new net N$26: IC5.-IN, R8.1, R9.2
- new net N$30: JP6.1, R24.2
- new net N$31: JP6.3, R32.2
- new net N$32: C36.2, Q3.1, U2.PB6(TOSC1/XTAL1)
- new net N$33: C37.1, Q3.2, U2.PB7(TOSC2/XTAL2)
- new net N$34: R37.1, R41.2
- new net N$35: R29.2, R41.1
- new net N$36: JP8-1.2, R40.2
- new net N$37: JP8-2.1, R38.2
- new net N$38: JP8-2.2, R37.2
- net +12V: now also C14.1, C28.1, IC4.V+, IC5.V+; no longer C1.1, C3.1, IC3.V+, IC6.V+
- net +3V3: now also C3.1, U1.OUT; no longer C25.1, IC2.OUT
- net +5V: now also C2.1, C31.1, C33.1, C35.2, JP7.1, JP8-1.1, LCD_POW.1, R29.1, R38.1, R40.1, R44.2, U$2.VCC, U1.IN, U2.AREF, U2.AVCC, U2.VCC; no longer C12.2, C26.1, C7.1, C9.1, IC2.IN, JP2.1, JP3-1.1, JP4.1, R13.1, R22.1, R26.1, R3.2, U$1.VCC, U1.AREF, U1.AVCC, U1.VCC
- net -12V: now also C21.2, C29.2, IC4.V-, IC5.V-; no longer C2.2, C4.2, IC3.V-, IC6.V-
- net A3: now also JP8-3.1, R28.2, U2.PC3(ADC3/PTCY); no longer JP3-3.1, R12.2, U1.PC3(ADC3/PTCY)
- net A4: now also JP8-3.2, R43.2, U2.PC4(ADC4/PTCY/SDA0); no longer JP3-3.2, R31.2, U1.PC4(ADC4/PTCY/SDA0)
- net A5: now also JP8-4.1, R42.2, U2.PC5(ADC5/PTCY/SCL0); no longer JP3-4.1, R30.2, U1.PC5(ADC5/PTCY/SCL0)
- net AGND: now also IC1.AGND, IC1.DGND, JP5.2; no longer X1.2
- net CS0: now also U2.PB2(PTCXY/OC1B/!SS0!); no longer U1.PB2(PTCXY/OC1B/!SS0!)
- net CS1: now also U2.PE2(ADC6/PTCY/ICP3/!SS1!); no longer U1.PE2(ADC6/PTCY/ICP3/!SS1!)
- net GAIN_OUT: now also IC4.OUT, R15.1; no longer IC3.OUT, R20.1
- net GND: now also C14.2, C2.2, C21.1, C28.2, C29.1, C32.1, C33.2, C34.2, C35.1, C36.1, C37.2, C40.2, JP6.2, LCD_POW.2, R28.1, R39.1, R42.1, R43.1, R7.1, R9.1, U$2.GND, U1.ADJ/GND, U2.1_GND, U2.2_GND; no longer C1.2, C10.2, C12.1, C13.2, C2.1, C22.1, C23.2, C25.2, C26.2, C4.1, C8.1, C9.2, IC1.AGND, IC1.DGND, IC2.ADJ, JP1.2, JP4.2, R12.1, R18.1, R23.1, R30.1, R31.1, R5.1, U$1.GND, U1.1_GND, U1.2_GND
- net MISO0: now also U$2.MISO, U2.PB4(PTCXY/RXD1/MISO0); no longer U$1.MISO, U1.PB4(PTCXY/RXD1/MISO0)
- net MOSI0: now also U$2.MOSI, U2.PB3(PTCXY/OC2A/TXD1/MOSI0); no longer U$1.MOSI, U1.PB3(PTCXY/OC2A/TXD1/MOSI0)
- net MOSI1: now also U2.PE3(ADC7/PTCY/T3/MOSI1); no longer U1.PE3(ADC7/PTCY/T3/MOSI1)
- net ROTA: now also C32.2, R32.1, U2.PD6(AIN0/PTCXY/OC0A); no longer C8.2, R16.1, U1.PD5(PTCXY/T1/OC0B)
- net ROTB: now also C34.1, R24.1, U2.PD5(PTCXY/T1/OC0B); no longer C10.1, R2.1, U1.PD6(AIN0/PTCXY/OC0A)
- net ROTBTN: now also C31.2, JP7.2, R39.2, U2.PD7(AIN1/PTCXY); no longer C7.2, JP2.2, R23.2, U1.PD7(AIN1/PTCXY)
- net SCK0: now also U$2.SCK, U2.PB5(PTCXY/XCK1/SCK0); no longer U$1.SCK, U1.PB5(PTCXY/XCK1/SCK0)
- net SCK1: now also U2.PC1(ADC1/PTCY/SCK1); no longer U1.PC1(ADC1/PTCY/SCK1)
- net SCL: now also LCD/I2C1.1, U2.PE1(PTCXY/T4/SCL1); no longer LCD/I2C.1, U1.PE1(PTCXY/T4/SCL1)
- net SDA: now also LCD/I2C1.2, U2.PE0(PTCXY/ACO/ICP4/SDA1); no longer LCD/I2C.2, U1.PE0(PTCXY/ACO/ICP4/SDA1)
- net SIG: now also R6.1; no longer R4.1
- net SIG_OUT: now also IC5.OUT, JP5.1, R8.2; no longer IC6.OUT, R17.2, X1.1
- net UC_RST: now also C40.1, R44.1, U$2.RST, U2.PC6(!RESET!); no longer C13.1, R3.1, U$1.RST, U1.PC6(!RESET!)
