File: funcgen.sch (EAGLE design)
At the start: 71 parts, among them IC1 AD9833, IC4 LM318D, IC5 LM318D, Q2 ASFL1, Q3 16MHz, U1 TLV1117-33IDCY, U2 MICROCHIP_ATMEGA328PB-AUMICRO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, U3 TLV61048DBVR

Commit message: Updated Board and Schematic
Updated Board and Schematic with SMA Schottky diodes and ISP pin 1 marking
Parts:
- removed D1, D2, D3: 1N5817-B, diode:1N5817-B
- added D4, D5, D6: MBR0520LT, diode:MBR0520LT
Connections:
- net +12V: now also D5.C; no longer D1.C
- net -12V: now also D6.A; no longer D2.A
- net N$11: now also D4.A, D6.C; no longer D2.C, D3.A
- net N$12: now also D4.C; no longer D3.C
- net N$9: now also D5.A; no longer D1.A
Changed lines of the file:
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@@
 <part name="R11" library="rcl" library_urn="urn:adsk.eagle:library:334" deviceset="R-EU_" device="R0805" package3d_urn="urn:adsk.eagle:package:23553/2" value="68k"/>
 <part name="U3" library="TLV61048DBVR" deviceset="TLV61048DBVR" device=""/>
-<part name="D1" library="diode" library_urn="urn:adsk.eagle:library:210" deviceset="1N581*" device="" package3d_urn="urn:adsk.eagle:package:43421/1" technology="7-B"/>
-<part name="D2" library="diode" library_urn="urn:adsk.eagle:library:210" deviceset="1N581*" device="" package3d_urn="urn:adsk.eagle:package:43421/1" technology="7-B"/>
-<part name="D3" library="diode" library_urn="urn:adsk.eagle:library:210" deviceset="1N581*" device="" package3d_urn="urn:adsk.eagle:package:43421/1" technology="7-B"/>
 <part name="GND8" library="supply1" library_urn="urn:adsk.eagle:library:371" deviceset="GND" device=""/>
 <part name="GND9" library="supply1" library_urn="urn:adsk.eagle:library:371" deviceset="GND" device=""/>
@@
 <part name="L1" library="rcl_2" deviceset="L-US" device="L0805" package3d_urn="urn:adsk.eagle:package:23617/2" value="4.7uH"/>
 <part name="JP1" library="jumper" library_urn="urn:adsk.eagle:library:252" deviceset="JP1E" device="" package3d_urn="urn:adsk.eagle:package:15455/1"/>
+<part name="D4" library="diode" library_urn="urn:adsk.eagle:library:210" deviceset="MBR0520LT" device="" package3d_urn="urn:adsk.eagle:package:43420/1"/>
+<part name="D5" library="diode" library_urn="urn:adsk.eagle:library:210" deviceset="MBR0520LT" device="" package3d_urn="urn:adsk.eagle:package:43420/1"/>
+<part name="D6" library="diode" library_urn="urn:adsk.eagle:library:210" deviceset="MBR0520LT" device="" package3d_urn="urn:adsk.eagle:package:43420/1"/>
 </parts>
 <sheets>
@@
 <attribute name="VALUE" x="137.16" y="138.24" size="2.0828" layer="96" ratio="10" rot="SR0"/>
 </instance>
-<instance part="D1" gate="G$1" x="177.8" y="170.18" smashed="yes">
-<attribute name="NAME" x="175.514" y="172.085" size="1.778" layer="95"/>
-<attribute name="VALUE" x="175.514" y="166.751" size="1.778" layer="96"/>
-</instance>
-<instance part="D2" gate="G$1" x="205.74" y="187.96" smashed="yes" rot="R180">
-<attribute name="NAME" x="208.026" y="186.055" size="1.778" layer="95" rot="R180"/>
-<attribute name="VALUE" x="208.026" y="191.389" size="1.778" layer="96" rot="R180"/>
-</instance>
-<instance part="D3" gate="G$1" x="205.74" y="180.34" smashed="yes">
-<attribute name="NAME" x="203.454" y="182.245" size="1.778" layer="95"/>
-<attribute name="VALUE" x="203.454" y="176.911" size="1.778" layer="96"/>
-</instance>
 <instance part="GND8" gate="1" x="170.18" y="142.24" smashed="yes">
 <attribute name="VALUE" x="167.64" y="139.7" size="1.778" layer="96"/>
@@
 <attribute name="NAME" x="38.1" y="207.01" size="1.778" layer="95" rot="R180"/>
 <attribute name="VALUE" x="38.1" y="213.995" size="1.778" layer="96" rot="R180"/>
+</instance>
+<instance part="D4" gate="G$1" x="205.74" y="180.34" smashed="yes">
+<attribute name="NAME" x="208.28" y="180.8226" size="1.778" layer="95"/>
+<attribute name="VALUE" x="208.28" y="178.0286" size="1.778" layer="96"/>
+</instance>
+<instance part="D5" gate="G$1" x="177.8" y="170.18" smashed="yes">
+<attribute name="NAME" x="180.34" y="170.6626" size="1.778" layer="95"/>
+<attribute name="VALUE" x="180.34" y="167.8686" size="1.778" layer="96"/>
+</instance>
+<instance part="D6" gate="G$1" x="205.74" y="187.96" smashed="yes" rot="R180">
+<attribute name="NAME" x="203.2" y="187.4774" size="1.778" layer="95" rot="R180"/>
+<attribute name="VALUE" x="203.2" y="190.2714" size="1.778" layer="96" rot="R180"/>
 </instance>
 </instances>
@@
 <pinref part="R1" gate="G$1" pin="1"/>
 <pinref part="U3" gate="G$1" pin="SW"/>
-<pinref part="D1" gate="G$1" pin="A"/>
 <wire x1="170.18" y1="180.34" x2="177.8" y2="180.34" width="0.1524" layer="91"/>
 <wire x1="167.64" y1="170.18" x2="170.18" y2="170.18" width="0.1524" layer="91"/>
@@
 <junction x="170.18" y="180.34"/>
 <pinref part="L1" gate="G$1" pin="2"/>
+<pinref part="D5" gate="G$1" pin="A"/>
 </segment>
 </net>
@@
 <segment>
 <pinref part="C18" gate="G$1" pin="2"/>
-<pinref part="D3" gate="G$1" pin="A"/>
 <wire x1="198.12" y1="180.34" x2="200.66" y2="180.34" width="0.1524" layer="91"/>
-<pinref part="D2" gate="G$1" pin="C"/>
 <wire x1="200.66" y1="180.34" x2="203.2" y2="180.34" width="0.1524" layer="91"/>
 <wire x1="203.2" y1="187.96" x2="200.66" y2="187.96" width="0.1524" layer="91"/>
 <wire x1="200.66" y1="187.96" x2="200.66" y2="180.34" width="0.1524" layer="91"/>
 <junction x="200.66" y="180.34"/>
+<pinref part="D6" gate="G$1" pin="C"/>
+<pinref part="D4" gate="G$1" pin="A"/>
 </segment>
 </net>
 <net name="N$12" class="0">
 <segment>
-<pinref part="D3" gate="G$1" pin="C"/>
 <pinref part="C19" gate="G$1" pin="2"/>
 <wire x1="208.28" y1="180.34" x2="215.9" y2="180.34" width="0.1524" layer="91"/>
+<pinref part="D4" gate="G$1" pin="C"/>
 </segment>
 </net>
@@
 <segment>
 <pinref part="C19" gate="G$1" pin="1"/>
-<pinref part="D2" gate="G$1" pin="A"/>
 <wire x1="215.9" y1="187.96" x2="208.28" y2="187.96" width="0.1524" layer="91"/>
 <pinref part="P-1" gate="1" pin="-12V"/>
 <wire x1="215.9" y1="187.96" x2="228.6" y2="187.96" width="0.1524" layer="91"/>
 <junction x="215.9" y="187.96"/>
+<pinref part="D6" gate="G$1" pin="A"/>
 </segment>
 </net>
 <net name="+12V" class="0">
 <segment>
-<pinref part="D1" gate="G$1" pin="C"/>
 <pinref part="R10" gate="G$1" pin="2"/>
 <wire x1="180.34" y1="170.18" x2="187.96" y2="170.18" width="0.1524" layer="91"/>
@@
 <wire x1="198.12" y1="170.18" x2="205.74" y2="170.18" width="0.1524" layer="91"/>
 <junction x="198.12" y="170.18"/>
-</segment>
-</net>
+<pinref part="D5" gate="G$1" pin="C"/>
+</segment>
+</net>
